File: macrofoob.kicad_pcb (KiCad board)
At the start: 2 copper layers, 373.7 x 104.5 mm, 115 parts, among them J1 SSD1306 128x32 OLED, Q1 2N 2222A, SW1 Switch, SW10 Switch, SW11 Switch, SW12 Switch, SW13 Switch, SW14 Switch, SW15 Switch, SW16 Switch, SW17 Switch, SW18 Switch, SW19 Switch, SW2 Switch, SW20 Switch, SW21 Switch, SW22 Switch, SW23 Switch, SW24 Switch, SW25 Switch, SW26 SW_Reset, SW3 Switch, SW4 Switch, SW5 Switch, SW6 Switch, SW7 Switch, SW8 Switch, SW9 Switch, U1 ProMicro

Commit message: added new TQFP-44 footprint with shorter pads
Other:
- net class Default: clearance 0.2 -> 0.25; via_dia 0.8 -> 1; via_drill 0.4 -> 0.6
- rule trace_clearance: 0.2 -> 0.25
Changed lines of the file:
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@@
   (setup
     (last_trace_width 0.25)
-    (trace_clearance 0.2)
+    (trace_clearance 0.25)
     (zone_clearance 0.508)
     (zone_45_only no)
     (trace_min 0.2)
-    (via_size 0.8)
-    (via_drill 0.4)
+    (via_size 1)
+    (via_drill 0.6)
     (via_min_size 0.4)
     (via_min_drill 0.3)
@@
     (pcb_text_width 0.3)
     (pcb_text_size 1.5 1.5)
-    (mod_edge_width 0.12)
+    (mod_edge_width 0.153)
     (mod_text_size 1 1)
-    (mod_text_width 0.15)
+    (mod_text_width 0.153)
     (pad_size 1.524 1.524)
     (pad_drill 0.762)
@@
   (net 63 "Net-(SW26-Pad1)")
   (net_class Default "This is the default net class."
-    (clearance 0.2)
+    (clearance 0.25)
     (trace_width 0.25)
-    (via_dia 0.8)
-    (via_drill 0.4)
+    (via_dia 1)
+    (via_drill 0.6)
     (uvia_dia 0.3)
     (uvia_drill 0.1)
+    (diff_pair_width 0.22)
+    (diff_pair_gap 0.165)
     (add_net +5V)
     (add_net COL1)

Commit message: initial pcb layout and schematic optimizations
Parts:
- removed the REF** at (352.3, 45.0)
- removed the REF** at (335.8, 97.0)
- removed the REF** at (354.8, 97.0)
- removed the REF** at (392.9, 97.0)
- removed the REF** at (316.7, 97.0)
- removed the REF** at (392.9, 78.0)
- removed the REF** at (354.8, 78.0)
- removed the REF** at (335.8, 78.0)
- removed the REF** at (373.9, 78.0)
- removed the REF** at (316.7, 78.0)
- removed the REF** at (392.9, 58.9)
- removed the REF** at (76.2, 30.3)
- removed the REF** at (354.8, 58.9)
- removed the REF** at (335.8, 58.9)
- removed the REF** at (373.9, 58.9)
- removed the REF** at (316.7, 58.9)
- removed the REF** at (392.9, 39.9)
- removed the REF** at (373.9, 39.9)
- removed the REF** at (335.8, 39.9)
- removed the REF** at (316.7, 39.9)
- removed the REF** at (344.7, 74.9)
- removed the REF** at (354.8, 116.1)
- removed the REF** at (392.9, 116.1)
- removed the REF** at (373.9, 116.1)
- removed the REF** at (316.7, 116.1)
- removed the REF** at (335.8, 116.1)
- removed the REF** at (373.9, 97.0)
- added C13: 0.1 uF, Capacitor_SMD:C_0805_2012Metric, F.Cu at (240.7, 53.2)
- added C14: 0.1 uF, Capacitor_SMD:C_0805_2012Metric, F.Cu at (245.1, 56.1)
- added C15: 0.1 uF, Capacitor_SMD:C_0805_2012Metric, F.Cu at (239.0, 59.1)
- added C16: 0.1 uF, Capacitor_SMD:C_0805_2012Metric, F.Cu at (249.5, 50.2)
- added C17: 1 uF, Capacitor_SMD:C_0805_2012Metric, F.Cu at (245.1, 53.2)
- added C18: 22 pF, Capacitor_SMD:C_0805_2012Metric, F.Cu at (249.5, 47.3)
- added C19: 22 pF, Capacitor_SMD:C_0805_2012Metric, F.Cu at (240.7, 56.1)
- added C20: 0.1 uF, Capacitor_SMD:C_0805_2012Metric, F.Cu at (245.1, 50.2)
- added C21: 1 uF, Capacitor_SMD:C_0805_2012Metric, F.Cu at (230.2, 58.9)
- added C22: 0.1 uF, Capacitor_SMD:C_0805_2012Metric, F.Cu at (201.8, 39.4)
- added C23: 0.1 uF, Capacitor_SMD:C_0805_2012Metric, F.Cu at (190.4, 44.4)
- added C24: 0.1 uF, Capacitor_SMD:C_0805_2012Metric, F.Cu at (176.4, 57.5)
- added C25: 0.1 uF, Capacitor_SMD:C_0805_2012Metric, F.Cu at (169.4, 64.1)
- added C26: 0.1 uF, Capacitor_SMD:C_0805_2012Metric, F.Cu at (169.4, 67.1)
- added C27: 0.1 uF, Capacitor_SMD:C_0805_2012Metric, F.Cu at (176.4, 54.5)
- added C28: 0.1 uF, Capacitor_SMD:C_0805_2012Metric, F.Cu at (173.8, 60.4)
- added C29: 0.1 uF, Capacitor_SMD:C_0805_2012Metric, F.Cu at (183.4, 52.4)
- added C30: 0.1 uF, Capacitor_SMD:C_0805_2012Metric, F.Cu at (187.8, 49.5)
- added C31: 0.1 uF, Capacitor_SMD:C_0805_2012Metric, F.Cu at (173.8, 63.4)
- added C32: 0.1 uF, Capacitor_SMD:C_0805_2012Metric, F.Cu at (194.8, 44.4)
- added C33: 0.1 uF, Capacitor_SMD:C_0805_2012Metric, F.Cu at (180.8, 55.4)
- added C34: 0.1 uF, Capacitor_SMD:C_0805_2012Metric, F.Cu at (178.2, 60.4)
- added C35: 0.1 uF, Capacitor_SMD:C_0805_2012Metric, F.Cu at (197.4, 39.4)
- added C36: 0.1 uF, Capacitor_SMD:C_0805_2012Metric, F.Cu at (178.2, 63.4)
- added C37: 0.1 uF, Capacitor_SMD:C_0805_2012Metric, F.Cu at (199.2, 42.3)
- added C38: 0.1 uF, Capacitor_SMD:C_0805_2012Metric, F.Cu at (192.2, 50.3)
- added C39: 0.1 uF, Capacitor_SMD:C_0805_2012Metric, F.Cu at (182.6, 58.3)
- added C40: 0.1 uF, Capacitor_SMD:C_0805_2012Metric, F.Cu at (182.6, 61.3)
- added C41: 0.1 uF, Capacitor_SMD:C_0805_2012Metric, F.Cu at (196.6, 47.4)
- added C42: 0.1 uF, Capacitor_SMD:C_0805_2012Metric, F.Cu at (185.2, 55.4)
- added C43: 0.1 uF, Capacitor_SMD:C_0805_2012Metric, F.Cu at (187.0, 58.3)
- added C44: 0.1 uF, Capacitor_SMD:C_0805_2012Metric, F.Cu at (206.3, 39.4)
- added C45: 0.1 uF, Capacitor_SMD:C_0805_2012Metric, F.Cu at (173.8, 66.3)
- added C46: 0.1 uF, Capacitor_SMD:C_0805_2012Metric, F.Cu at (187.8, 52.4)
- added D27: D_TVS, Diode_SMD:D_SMA, F.Cu at (216.4, 54.6)
- added D28: D_TVS, Diode_SMD:D_SMA, F.Cu at (241.5, 40.2)
- added D29: D_TVS, Diode_SMD:D_SMA, F.Cu at (216.4, 59.2)
- added F1: Polyfuse 500 mA, Fuse:Fuse_1812_4532Metric, F.Cu at (249.0, 40.4)
- added J2: ISP Header, Connector_PinHeader_2.54mm:PinHeader_2x03_P2.54mm_Vertical, F.Cu at (229.2, 50.0)
- added J3: SSD1306 128x32 OLED, Connector_PinHeader_2.54mm:PinHeader_1x04_P2.54mm_Vertical, F.Cu at (158.4, 74.9)
- added J4: POWER, testatur:Generic_Pads_2mm_1x2, F.Cu at (186.7, 97.2)
- added J5: I2C, testatur:Generic_Pads_2mm_1x2, F.Cu at (183.7, 97.2)
- added J6: MATRIX_COLUMNS, testatur:Generic_Pads_2mm_1x5, F.Cu at (154.6, 74.1)
- added J7: MATRIX_ROWS, testatur:Generic_Pads_2mm_1x5, F.Cu at (154.6, 89.1)
- added J8: LED_DATA, testatur:Generic_Pads_2mm_1x1, F.Cu at (206.1, 83.5)
- added J9: LED_DATA, testatur:Generic_Pads_2mm_1x1, F.Cu at (199.6, 57.1)
- added LED13: ComboLED, testatur:LED_combined_SK6812MINI_0805, F.Cu at (76.2, 71.1)
- added LED14: ComboLED, testatur:LED_combined_SK6812MINI_0805, F.Cu at (95.2, 71.1)
- added LED15: ComboLED, testatur:LED_combined_SK6812MINI_0805, F.Cu at (114.3, 71.1)
- added LED16: ComboLED, testatur:LED_combined_SK6812MINI_0805, F.Cu at (38.1, 90.2)
- added LED17: ComboLED, testatur:LED_combined_SK6812MINI_0805, F.Cu at (57.1, 90.2)
- added LED18: ComboLED, testatur:LED_combined_SK6812MINI_0805, F.Cu at (76.2, 90.2)
- added LED19: ComboLED, testatur:LED_combined_SK6812MINI_0805, F.Cu at (95.2, 90.2)
- added LED20: ComboLED, testatur:LED_combined_SK6812MINI_0805, F.Cu at (114.3, 90.2)
- added LED21: ComboLED, testatur:LED_combined_SK6812MINI_0805_cutout, F.Cu at (38.1, 109.2)
- added LED22: ComboLED, testatur:LED_combined_SK6812MINI_0805, F.Cu at (57.1, 109.2)
- added LED23: ComboLED, testatur:LED_combined_SK6812MINI_0805, F.Cu at (76.2, 109.2)
- added LED24: ComboLED, testatur:LED_combined_SK6812MINI_0805, F.Cu at (95.2, 109.2)
- added LED25: ComboLED, testatur:LED_combined_SK6812MINI_0805_cutout, F.Cu at (114.3, 109.2)
- added LED26: SK6812MINI, LED_SMD:LED_SK6812MINI_PLCC4_3.5x3.5mm_P1.75mm, F.Cu at (183.0, 80.1)
- added LED27: SK6812MINI, LED_SMD:LED_SK6812MINI_PLCC4_3.5x3.5mm_P1.75mm, F.Cu at (159.6, 100.3)
- added LED28: SK6812MINI, LED_SMD:LED_SK6812MINI_PLCC4_3.5x3.5mm_P1.75mm, F.Cu at (159.6, 95.3)
- added LED29: SK6812MINI, LED_SMD:LED_SK6812MINI_PLCC4_3.5x3.5mm_P1.75mm, F.Cu at (166.6, 90.2)
- added LED30: SK6812MINI, LED_SMD:LED_SK6812MINI_PLCC4_3.5x3.5mm_P1.75mm, F.Cu at (168.9, 75.1)
- added LED31: SK6812MINI, LED_SMD:LED_SK6812MINI_PLCC4_3.5x3.5mm_P1.75mm, F.Cu at (175.9, 75.1)
- added LED32: SK6812MINI, LED_SMD:LED_SK6812MINI_PLCC4_3.5x3.5mm_P1.75mm, F.Cu at (159.6, 90.2)
- added LED33: SK6812MINI, LED_SMD:LED_SK6812MINI_PLCC4_3.5x3.5mm_P1.75mm, F.Cu at (171.3, 85.2)
- added LED34: SK6812MINI, LED_SMD:LED_SK6812MINI_PLCC4_3.5x3.5mm_P1.75mm, F.Cu at (164.3, 85.2)
- added LED35: SK6812MINI, LED_SMD:LED_SK6812MINI_PLCC4_3.5x3.5mm_P1.75mm, F.Cu at (175.9, 80.1)
- added LED36: SK6812MINI, LED_SMD:LED_SK6812MINI_PLCC4_3.5x3.5mm_P1.75mm, F.Cu at (168.9, 80.1)
- added LED37: SK6812MINI, LED_SMD:LED_SK6812MINI_PLCC4_3.5x3.5mm_P1.75mm, F.Cu at (183.0, 75.1)
- added LED38: LED, LED_SMD:LED_0805_2012Metric, F.Cu at (239.7, 44.0)
- added NT1: Net-Tie_2, NetTie:NetTie-2_SMD_Pad2.0mm, F.Cu at (224.2, 59.2)
- added Q2: Q_NMOS_GSD, Package_TO_SOT_SMD:SOT-23, F.Cu at (169.4, 60.4)
- added R10: 4.7k, Resistor_SMD:R_0805_2012Metric, F.Cu at (244.1, 44.3)
- added R11: 500, Resistor_SMD:R_0805_2012Metric, F.Cu at (236.2, 52.1)
- added R12: 470, Resistor_SMD:R_0805_2012Metric, F.Cu at (192.2, 53.3)
- added R13: 470, Resistor_SMD:R_0805_2012Metric, F.Cu at (205.4, 48.2)
- added R14: 470, Resistor_SMD:R_0805_2012Metric, F.Cu at (203.7, 42.3)
- added R15: 470, Resistor_SMD:R_0805_2012Metric, F.Cu at (196.6, 50.3)
- added R16: 470, Resistor_SMD:R_0805_2012Metric, F.Cu at (182.6, 64.2)
- added R17: 470, Resistor_SMD:R_0805_2012Metric, F.Cu at (187.0, 61.3)
- added R18: 470, Resistor_SMD:R_0805_2012Metric, F.Cu at (201.0, 45.3)
- added R19: 470, Resistor_SMD:R_0805_2012Metric, F.Cu at (178.2, 66.3)
- added R20: 470, Resistor_SMD:R_0805_2012Metric, F.Cu at (183.4, 49.5)
- added R21: 470, Resistor_SMD:R_0805_2012Metric, F.Cu at (201.0, 48.2)
- added R22: 470, Resistor_SMD:R_0805_2012Metric, F.Cu at (182.6, 67.2)
- added R23: 470, Resistor_SMD:R_0805_2012Metric, F.Cu at (196.6, 53.3)
- added R24: 470, Resistor_SMD:R_0805_2012Metric, F.Cu at (191.4, 59.2)
- added R25: 470, Resistor_SMD:R_0805_2012Metric, F.Cu at (205.4, 45.3)
- added R26: 470, Resistor_SMD:R_0805_2012Metric, F.Cu at (187.0, 64.2)
- added R27: 470, Resistor_SMD:R_0805_2012Metric, F.Cu at (201.0, 51.2)
- added R28: 470, Resistor_SMD:R_0805_2012Metric, F.Cu at (195.9, 56.2)
- added R29: 470, Resistor_SMD:R_0805_2012Metric, F.Cu at (191.4, 56.2)
- added R30: 470, Resistor_SMD:R_0805_2012Metric, F.Cu at (192.2, 47.4)
- added R31: 470, Resistor_SMD:R_0805_2012Metric, F.Cu at (191.4, 62.1)
- added R32: 470, Resistor_SMD:R_0805_2012Metric, F.Cu at (187.0, 67.2)
- added R33: 470, Resistor_SMD:R_0805_2012Metric, F.Cu at (195.9, 59.2)
- added R34: 470, Resistor_SMD:R_0805_2012Metric, F.Cu at (201.0, 54.1)
- added R35: 470, Resistor_SMD:R_0805_2012Metric, F.Cu at (205.4, 51.2)
- added R36: 470, Resistor_SMD:R_0805_2012Metric, F.Cu at (191.4, 65.1)
- added R37: 1k, Resistor_SMD:R_0805_2012Metric, F.Cu at (195.9, 62.1)
- added R5: 5.1k, Resistor_SMD:R_0805_2012Metric, B.Cu at (73.2, 35.9)
- added R6: 1k, Resistor_SMD:R_0805_2012Metric, F.Cu at (236.2, 49.2)
- added R7: 22, Resistor_SMD:R_0805_2012Metric, B.Cu at (69.1, 30.0)
- added R8: 22, Resistor_SMD:R_0805_2012Metric, B.Cu at (69.1, 32.0)
- added R9: 4.7k, Resistor_SMD:R_0805_2012Metric, F.Cu at (236.2, 55.1)
- added REF**: QFN-44-1EP_7x7mm_P0.5mm_EP5.2x5.2mm, Package_DFN_QFN:QFN-44-1EP_7x7mm_P0.5mm_EP5.2x5.2mm, B.Cu at (144.4, 32.9)
- added Y1: 16 MHz, Resistor_SMD:R_1210_3225Metric, F.Cu at (223.2, 54.5)
- D3, D4, D5, D6, D7, LS1, SW26: moved to F.Cu
- J1: value SSD1306 128x32 OLED -> USB_C_Receptacle; footprint Connector_PinHeader_2.54mm:PinHeader_1x04_P2.54mm_Vertical -> testatur:HRO-TYPE-C-31-M-12_kicad-pinout; moved to B.Cu
- LED1, LED5: value SK6812MINI -> ComboLED; footprint LED_SMD:LED_SK6812MINI_PLCC4_3.5x3.5mm_P1.75mm -> testatur:LED_combined_SK6812MINI_0805_cutout
- LED10, LED11, LED12, LED2, LED3, LED4, LED6, LED7, LED8, LED9: value SK6812MINI -> ComboLED; footprint LED_SMD:LED_SK6812MINI_PLCC4_3.5x3.5mm_P1.75mm -> testatur:LED_combined_SK6812MINI_0805
- R3: value 4.7k -> 5.1k
- R4: value 4.7k -> 5.1k; moved to B.Cu
- RC1, RC2, RC3, RC4: footprint testatur:RotaryEncoder_Alps_EC11E-Switch_Vertical_H20mm_custom -> testatur:RotaryEncoder_Alps_EC11E-Switch_Vertical_H20mm_custom_minimalpads
- U1: value ProMicro -> ATmega32U4-AU; footprint promicro:ProMicroModified -> testatur:TQFP-44_10x10mm_P0.8mm_short
- moved D26 268.7 mm to (196.0, 80.7)
- moved D22 262.2 mm to (179.7, 87.5)
- moved D24 261.0 mm to (196.0, 74.2)
- moved D13 259.2 mm to (186.0, 94.0)
- moved D25 251.3 mm to (184.3, 84.3)
- moved D8 241.3 mm to (202.3, 74.2)
- moved D17 235.0 mm to (190.7, 83.9)
- moved D12 230.5 mm to (192.4, 87.2)
- moved C11 227.8 mm to (202.4, 83.5)
- moved D11 226.2 mm to (197.0, 83.9)
- moved C1 226.2 mm to (201.4, 80.5)
- moved D23 224.8 mm to (173.1, 95.8)
- moved D9 224.6 mm to (202.3, 77.4)
- moved LED5 223.9 mm to (114.3, 33.0)
- moved D19 222.8 mm to (189.7, 80.7)
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Connections:
- C1 pad 1: +5V -> VCC
- C10 pad 1: +5V -> VCC
- C11 pad 1: +5V -> VCC
- C12 pad 1: +5V -> VCC
- C2 pad 1: +5V -> VCC
- C3 pad 1: +5V -> VCC
- C4 pad 1: +5V -> VCC
- C5 pad 1: +5V -> VCC
- C6 pad 1: +5V -> VCC
- C7 pad 1: +5V -> VCC
- C8 pad 1: +5V -> VCC
- C9 pad 1: +5V -> VCC
- LED1 pad 2: +5V -> GND
- LED1 pad 3: RGB_DIN -> Backlight_RGB
- LED1 pad 4: GND -> VCC
- LED10 pad 2: +5V -> GND
- LED10 pad 4: GND -> VCC
- LED11 pad 2: +5V -> GND
- LED11 pad 4: GND -> VCC
- LED12 pad 2: +5V -> GND
- LED12 pad 4: GND -> VCC
- LED2 pad 2: +5V -> GND
- LED2 pad 4: GND -> VCC
- LED3 pad 2: +5V -> GND
- LED3 pad 4: GND -> VCC
- LED4 pad 2: +5V -> GND
- LED4 pad 4: GND -> VCC
- LED5 pad 2: +5V -> GND
- LED5 pad 4: GND -> VCC
- LED6 pad 2: +5V -> GND
- LED6 pad 4: GND -> VCC
- LED7 pad 2: +5V -> GND
- LED7 pad 4: GND -> VCC
- LED8 pad 2: +5V -> GND
- LED8 pad 4: GND -> VCC
- LED9 pad 2: +5V -> GND
- LED9 pad 4: GND -> VCC
- LS1 pad 1: +5V -> VCC
- R1 pad 1: +5V -> VCC
- R3 pad 1: VCC -> Reset
- R3 pad 2: SDA -> VCC
- R4 pad 1: VCC -> GND
- R4 pad 2: SCL -> Net-(J1-PadA5)
- SW26 pad 1: Net-(SW26-Pad1) -> Reset
- SW26 pad 2: Net-(SW26-Pad2) -> GND
- U1 pad 1: RC2A -> Net-(U1-Pad1)
- U1 pad 10: COL5 -> MOSI
- U1 pad 11: COL4 -> MISO
- U1 pad 12: COL3 -> Backlight
- U1 pad 13: PIEZO -> Reset
- U1 pad 14: COL2 -> VCC
- U1 pad 15: COL1 -> GND
- U1 pad 16: ROW3 -> Net-(C19-Pad1)
- U1 pad 17: ROW4 -> Net-(C18-Pad1)
- U1 pad 18: ROW5 -> SCL
- U1 pad 19: RC1B -> SDA
- U1 pad 2: RC2B -> VCC
- U1 pad 20: RC1A -> RC2A
- U1 pad 21: VCC -> RC2B
- U1 pad 22: Net-(SW26-Pad2) -> ROW2
- U1 pad 23: Net-(SW26-Pad1) -> GND
- U1 pad 24: +5V -> VCC
- U1 pad 3: GND -> D-
- U1 pad 4: GND -> D+
- U1 pad 5: SCL -> GND
- U1 pad 6: SDA -> Net-(C21-Pad1)
- U1 pad 7: RGB_DIN -> VCC
- U1 pad 8: ROW2 -> Net-(R6-Pad2)
- U1 pad 9: ROW1 -> SCK
Routing:
- net ROW1: track 122.9 -> 0.00 mm, vias 5 -> 0
- net COL1: track 19.2 -> 0.00 mm
- net COL2: track 19.0 -> 0.00 mm
- net SW1: track 17.0 -> 0.00 mm
- net Net-(D4-Pad2): track 14.2 -> 0.00 mm
- net Net-(D3-Pad2): track 14.2 -> 0.00 mm
- net Net-(D2-Pad2): track 14.2 -> 0.00 mm
- net SW5: track 14.2 -> 0.00 mm
- net /MCU/Dcon+: track 0.00 -> 2.93 mm
- net /MCU/Dcon-: track 0.00 -> 2.93 mm
- net Net-(J1-PadA5): track 0.00 -> 2.31 mm
- net Net-(J1-PadB5): track 0.00 -> 2.11 mm
Other:
- board size 373.7 x 104.5 mm -> 100 x 100 mm
- net class Default: clearance 0.25 -> 0.2; trace_width 0.25 -> 0.2; via_dia 1 -> 0.6; via_drill 0.6 -> 0.3
- rule pad_to_mask_clearance: 0.051 -> 0.1
- rule solder_mask_min_width: 0.25 -> 0.2
- rule trace_clearance: 0.25 -> 0.2
